Commit message: Add gazebo_ros_control PID gains
Tuned manually to make movement via the teleop interface behave well
Wheels still unspecified because they cause the robot to collapse
Use effort joint interface for the gripper so that gripper contacts are well simulated
Make additional cameras massless to avoid interference with arm simulation. Needs to be double checked to ensure having zero mass doesn't cause its own simulation issues

File: robots/forky.gazebo.xacro (robot description, xacro)
@@ -32,7 +32,7 @@
     </visual>
     <inertial>
-      <mass value="1e-5" />
+      <mass value="0" />
       <origin xyz="0 0 0" rpy="0 0 0"/>
-      <inertia ixx="1e-6" ixy="0" ixz="0" iyy="1e-6" iyz="0" izz="1e-6" />
+      <inertia ixx="0" ixy="0" ixz="0" iyy="0" iyz="0" izz="0" />
     </inertial>
   </link>
@@ -62,7 +62,7 @@
     </visual>
     <inertial>
-      <mass value="1e-5" />
+      <mass value="0" />
       <origin xyz="0 0 0" rpy="0 0 0"/>
-      <inertia ixx="1e-6" ixy="0" ixz="0" iyy="1e-6" iyz="0" izz="1e-6" />
+      <inertia ixx="0" ixy="0" ixz="0" iyy="0" iyz="0" izz="0" />
     </inertial>
   </link>
@@ -683,5 +683,5 @@
     </actuator>
     <joint name="joint_gripper_finger_left">
-      <hardwareInterface>hardware_interface/PositionJointInterface</hardwareInterface>
+      <hardwareInterface>hardware_interface/EffortJointInterface</hardwareInterface>
     </joint>
   </transmission>
@@ -692,5 +692,5 @@
     </actuator>
     <joint name="joint_gripper_finger_right">
-      <hardwareInterface>hardware_interface/PositionJointInterface</hardwareInterface>
+      <hardwareInterface>hardware_interface/EffortJointInterface</hardwareInterface>
     </joint>
 </transmission>

Commit message: Fix misspecified materials on forky
Had been causing warnings when building the URDF

File: robots/forky.gazebo.xacro (robot description, xacro)
@@ -29,5 +29,7 @@
     <sphere radius="${camera_link}"/>
       </geometry>
-      <material name="gray"/>
+      <material name="">
+        <color rgba="0.1 0.1 0.1 1" />
+      </material>
     </visual>
     <inertial>
@@ -59,5 +61,7 @@
     <sphere radius="${camera_link}"/>
       </geometry>
-      <material name="gray"/>
+      <material name="">
+              <color rgba="0.1 0.1 0.1 1" />
+            </material>
     </visual>
     <inertial>

Commit message: Reformat some whitespace in launch and xacro files

File: robots/forky.gazebo.xacro (robot description, xacro)
@@ -10,5 +10,5 @@
   <xacro:include filename="$(find stretch_description)/urdf/stretch_respeaker.xacro" />
   <xacro:include filename="$(find stretch_description)/urdf/stretch_gripper.xacro" />
-<xacro:property name="camera_link" value="0.015" /> <!-- Size of square 'camera' box -->
+  <xacro:property name="camera_link" value="0.015" /> <!-- Size of square 'camera' box -->
   <!-- Navigation Camera -->
   <joint name="navigation_camera_joint" type="fixed">
@@ -40,7 +40,7 @@
     </inertial>
   </link>
-      <gazebo reference="navigation_camera_link">
-          <material>Gazebo/Black</material>
-      </gazebo>
+  <gazebo reference="navigation_camera_link">
+      <material>Gazebo/Black</material>
+  </gazebo>
   <!-- Gripper Camera -->
   <joint name="gripper_camera_joint" type="fixed">
@@ -141,5 +141,5 @@
         <clip>
           <near>0.02</near>
-          <far>300</far>
+          <far>100</far>
         </clip>
         <noise>
@@ -168,44 +168,44 @@
     </sensor>
   </gazebo>
-    <!-- Gripper camera -->
-      <gazebo reference="gripper_camera_link">
-        <sensor type="camera" name="gripper_camera">
-          <update_rate>6.0</update_rate>
-          <camera name="head">
-            <horizontal_fov>1.8</horizontal_fov>
-            <image>
-              <width>1024</width>
-              <height>768</height>
-              <format>R8G8B8</format>
-            </image>
-            <clip>
-              <near>0.02</near>
-              <far>300</far>
-            </clip>
-            <noise>
-              <type>gaussian</type>
-              <!-- Noise is sampled independently per pixel on each frame.
-                   That pixel's noise value is added to each of its color
-                   channels, which at that point lie in the range [0,1]. -->
-              <mean>0.0</mean>
-              <stddev>0.007</stddev>
-            </noise>
-          </camera>
-          <plugin name="camera_controller" filename="libgazebo_ros_camera.so">
-            <alwaysOn>false</alwaysOn>
-            <updateRate>0.0</updateRate>
-            <cameraName>gripper_camera</cameraName>
-            <imageTopicName>image_raw</imageTopicName>
-            <cameraInfoTopicName>camera_info</cameraInfoTopicName>
-            <frameName>camera_link</frameName>
-            <hackBaseline>0.07</hackBaseline>
-            <distortionK1>0.0</distortionK1>
-            <distortionK2>0.0</distortionK2>
-            <distortionK3>0.0</distortionK3>
-            <distortionT1>0.0</distortionT1>
-            <distortionT2>0.0</distortionT2>
-          </plugin>
-        </sensor>
-      </gazebo>
+  <!-- Gripper camera -->
+  <gazebo reference="gripper_camera_link">
+    <sensor type="camera" name="gripper_camera">
+      <update_rate>6.0</update_rate>
+      <camera name="head">
+        <horizontal_fov>1.8</horizontal_fov>
+        <image>
+          <width>1024</width>
+          <height>768</height>
+          <format>R8G8B8</format>
+        </image>
+        <clip>
+          <near>0.02</near>
+          <far>100</far>
+        </clip>
+        <noise>
+          <type>gaussian</type>
+          <!-- Noise is sampled independently per pixel on each frame.
+               That pixel's noise value is added to each of its color
+               channels, which at that point lie in the range [0,1]. -->
+          <mean>0.0</mean>
+          <stddev>0.007</stddev>
+        </noise>
+      </camera>
+      <plugin name="camera_controller" filename="libgazebo_ros_camera.so">
+        <alwaysOn>false</alwaysOn>
+        <updateRate>0.0</updateRate>
+        <cameraName>gripper_camera</cameraName>
+        <imageTopicName>image_raw</imageTopicName>
+        <cameraInfoTopicName>camera_info</cameraInfoTopicName>
+        <frameName>camera_link</frameName>
+        <hackBaseline>0.07</hackBaseline>
+        <distortionK1>0.0</distortionK1>
+        <distortionK2>0.0</distortionK2>
+        <distortionK3>0.0</distortionK3>
+        <distortionT1>0.0</distortionT1>
+        <distortionT2>0.0</distortionT2>
+      </plugin>
+    </sensor>
+  </gazebo>
   <xacro:if value="${'$(arg realsense)' == 'false' }">
     <gazebo reference="camera_depth_frame">
@@ -744,5 +744,5 @@
       <hardwareInterface>hardware_interface/EffortJointInterface</hardwareInterface>
     </joint>
-</transmission>
+  </transmission>
 <!-- Ground Truth Odom plugin -->
   <!-- Ground Truth Odom plugin -->

Commit message: Add dexwrist support, better materials, and camera distortion
Add speculative attachment point for gripper camera alognside dexwrist
Add color-matched materials
Distortion is manually tuned to get the same crazy vignetting, but these will need additional cropping to better represent the real cameras
Add mimic joint plugin to gripper and arm to correctly sync joints

File: robots/forky.gazebo.xacro (robot description, xacro)
@@ -1,7 +1,9 @@
 <?xml version="1.0"?>
-<robot xmlns:xacro="http://www.ros.org/wiki/xacro" name="stretch_description">
+<robot xmlns:xacro="http://www.ros.org/wiki/xacro" name="forky">
   <xacro:arg name="gpu_lidar" default="false" />
   <xacro:arg name="visualize_lidar" default="false" />
   <xacro:arg name="realsense" default="true" />
+  <xacro:arg name="tool" default="gripper" />
+  <xacro:arg name="fisheyes" default="true" />
   <xacro:include filename="$(find stretch_description)/urdf/stretch_main.xacro" />
   <xacro:include filename="$(find stretch_description)/urdf/stretch_aruco.xacro" />
@@ -9,70 +11,173 @@
   <xacro:include filename="$(find stretch_description)/urdf/stretch_laser_range_finder.xacro" />
   <xacro:include filename="$(find stretch_description)/urdf/stretch_respeaker.xacro" />
-  <xacro:include filename="$(find stretch_description)/urdf/stretch_gripper.xacro" />
-  <xacro:property name="camera_link" value="0.015" /> <!-- Size of square 'camera' box -->
-  <!-- Navigation Camera -->
-  <joint name="navigation_camera_joint" type="fixed">
-    <axis xyz="0 1 0" />
-    <origin xyz="0 .125 -0.01" rpy="0 1.57 0"/>
-    <parent link="link_head"/>
-    <child link="navigation_camera_link"/>
-  </joint>
-  <link name="navigation_camera_link">
-    <collision>
-      <origin xyz="0 0 0" rpy="0 0 0"/>
-      <geometry>
-    <sphere radius="${camera_link}"/>
-      </geometry>
-    </collision>
-    <visual>
-      <origin xyz="0 0 0" rpy="0 0 0"/>
-      <geometry>
-    <sphere radius="${camera_link}"/>
-      </geometry>
-      <material name="">
-        <color rgba="0.1 0.1 0.1 1" />
-      </material>
-    </visual>
-    <inertial>
-      <mass value="0" />
-      <origin xyz="0 0 0" rpy="0 0 0"/>
-      <inertia ixx="0" ixy="0" ixz="0" iyy="0" iyz="0" izz="0" />
-    </inertial>
-  </link>
-  <gazebo reference="navigation_camera_link">
-      <material>Gazebo/Black</material>
-  </gazebo>
-  <!-- Gripper Camera -->
-  <joint name="gripper_camera_joint" type="fixed">
-    <axis xyz="0 1 0" />
-    <origin xyz="-.125 0 -.05 " rpy="0 .7 3.14"/>
-    <parent link="link_gripper"/>
-    <child link="gripper_camera_link"/>
-  </joint>
-  <link name="gripper_camera_link">
-    <collision>
-      <origin xyz="0 0 0" rpy="0 0 0"/>
-      <geometry>
-    <sphere radius="${camera_link}"/>
-      </geometry>
-    </collision>
-    <visual>
-      <origin xyz="0 0 0" rpy="0 0 0"/>
-      <geometry>
-    <sphere radius="${camera_link}"/>
-      </geometry>
-      <material name="">
-              <color rgba="0.1 0.1 0.1 1" />
-            </material>
-    </visual>
-    <inertial>
-      <mass value="0" />
-      <origin xyz="0 0 0" rpy="0 0 0"/>
-      <inertia ixx="0" ixy="0" ixz="0" iyy="0" iyz="0" izz="0" />
-    </inertial>
-  </link>
+  <xacro:if value="${'$(arg tool)' == 'gripper' }">
+    <xacro:include filename="$(find hcrl_gazebo)/urdf/stretch_gripper.gazebo.xacro" />
+    <xacro:stretch-gripper-gazebo/>
+  </xacro:if>
+  <xacro:if value="${'$(arg tool)' == 'dex_wrist' }">
+    <xacro:include filename="$(find hcrl_gazebo)/urdf/stretch_dex_wrist.gazebo.xacro" />
+    <xacro:stretch-dex-wrist-gazebo/>
+  </xacro:if>
+  <xacro:if value="${'$(arg fisheyes)' == 'true' }">
+      <xacro:property name="camera_link" value="0.015" /> <!-- Size of square 'camera' box -->
+    <!-- Navigation Camera -->
+    <joint name="navigation_camera_joint" type="fixed">
+      <axis xyz="0 1 0" />
+      <origin xyz="0 .125 -0.01" rpy="0 1.57 0"/>
+      <parent link="link_head"/>
+      <child link="navigation_camera_link"/>
+    </joint>
+    <link name="navigation_camera_link">
+      <collision>
+        <origin xyz="0 0 0" rpy="0 0 0"/>
+        <geometry>
+      <sphere radius="${camera_link}"/>
+        </geometry>
+      </collision>
+      <visual>
+        <origin xyz="0 0 0" rpy="0 0 0"/>
+        <geometry>
+      <sphere radius="${camera_link}"/>
+        </geometry>
+        <material name="">
+          <color rgba="0.1 0.1 0.1 1" />
+        </material>
+      </visual>
+      <inertial>
+        <mass value="0" />
+        <origin xyz="0 0 0" rpy="0 0 0"/>
+        <inertia ixx="0" ixy="0" ixz="0" iyy="0" iyz="0" izz="0" />
+      </inertial>
+    </link>
+    <gazebo reference="navigation_camera_link">
+        <material>HelloRobot/Black</material>
+    </gazebo>
+    <!-- Gripper Camera -->
+    <xacro:if value="${'$(arg tool)' == 'gripper' }">
+      <joint name="gripper_camera_joint" type="fixed">
+        <axis xyz="0 1 0" />
+        <origin xyz="-.125 0 -.05 " rpy="0 .7 3.14"/>
+        <parent link="link_gripper"/>
+        <child link="gripper_camera_link"/>
+      </joint>
+    </xacro:if>
+    <xacro:if value="${'$(arg tool)' == 'dex_wrist' }">
+      <joint name="gripper_camera_joint" type="fixed">
+        <axis xyz="0 1 0" />
+        <origin xyz="-.125 0 -.05 " rpy="0 .7 3.14"/>
+        <parent link="link_wrist_yaw"/>
+        <child link="gripper_camera_link"/>
+      </joint>
+    </xacro:if>
+    <link name="gripper_camera_link">
+      <collision>
+        <origin xyz="0 0 0" rpy="0 0 0"/>
+        <geometry>
+      <sphere radius="${camera_link}"/>
+        </geometry>
+      </collision>
+      <visual>
+        <origin xyz="0 0 0" rpy="0 0 0"/>
+        <geometry>
+      <sphere radius="${camera_link}"/>
+        </geometry>
+        <material name="">
+                <color rgba="0.1 0.1 0.1 1" />
+              </material>
+      </visual>
+      <inertial>
+        <mass value="0" />
+        <origin xyz="0 0 0" rpy="0 0 0"/>
+        <inertia ixx="0" ixy="0" ixz="0" iyy="0" iyz="0" izz="0" />
+      </inertial>
+    </link>
     <gazebo reference="gripper_camera_link">
-        <material>Gazebo/Black</material>
-    </gazebo>
+        <material>HelloRobot/Black</material>
+    </gazebo>
+    <!-- Navigation camera -->
+    <gazebo reference="navigation_camera_link">
+      <sensor name="navigation_camera" type="wideanglecamera">
+        <camera>
+          <horizontal_fov>2.55</horizontal_fov>
+          <image>
+            <width>1024</width>
+            <height>768</height>
+          </image>
+          <clip>
+            <near>0.01</near>
+            <far>100</far>
+          </clip>
+          <lens>
+            <type>custom</type>
+            <custom_function>
+              <c1>1.05</c1>
+              <c2>4</c2>
+              <f>1.0</f>
+              <fun>tan</fun>
+            </custom_function>
+            <cutoff_angle>1.3</cutoff_angle>
+          </lens>
+          <always_on>1</always_on>
+          <update_rate>6</update_rate>
+        </camera>
+        <plugin name="camera_controller" filename="libgazebo_ros_camera.so">
+          <alwaysOn>false</alwaysOn>
+          <updateRate>0.0</updateRate>
+          <cameraName>navigation_camera</cameraName>
+          <imageTopicName>image_raw</imageTopicName>
+          <cameraInfoTopicName>camera_info</cameraInfoTopicName>
+          <frameName>camera_link</frameName>
+          <hackBaseline>0.07</hackBaseline>
+          <distortionK1>0.0</distortionK1>
+          <distortionK2>0.0</distortionK2>
+          <distortionK3>0.0</distortionK3>
+          <distortionT1>0.0</distortionT1>
+          <distortionT2>0.0</distortionT2>
+        </plugin>
+      </sensor>
+    </gazebo>
+    <!-- Gripper camera -->
+    <gazebo reference="gripper_camera_link">
+      <sensor name="gripper_camera" type="wideanglecamera">
+        <camera>
+          <horizontal_fov>2.55</horizontal_fov>
+          <image>
+            <width>1024</width>
+            <height>768</height>
+          </image>
+          <clip>
+            <near>0.01</near>
+            <far>100</far>
+          </clip>
+          <lens>
+            <type>custom</type>
+            <custom_function>
+              <c1>1.05</c1>
+              <c2>4</c2>
+              <f>1.0</f>
+              <fun>tan</fun>
+            </custom_function>
+            <cutoff_angle>1.3</cutoff_angle>
+          </lens>
+          <always_on>1</always_on>
+          <update_rate>6</update_rate>
+        </camera>
+        <plugin name="camera_controller" filename="libgazebo_ros_camera.so">
+          <alwaysOn>false</alwaysOn>
+          <updateRate>0.0</updateRate>
+          <cameraName>gripper_camera</cameraName>
+          <imageTopicName>image_raw</imageTopicName>
+          <cameraInfoTopicName>camera_info</cameraInfoTopicName>
+          <frameName>camera_link</frameName>
+          <hackBaseline>0.07</hackBaseline>
+          <distortionK1>0.0</distortionK1>
+          <distortionK2>0.0</distortionK2>
+          <distortionK3>0.0</distortionK3>
+          <distortionT1>0.0</distortionT1>
+          <distortionT2>0.0</distortionT2>
+        </plugin>
+      </sensor>
+    </gazebo>
+  </xacro:if>
   <gazebo>
     <plugin name="gazebo_ros_control" filename="libhcrl_gazebo_ros_control_plugin.so">
@@ -84,5 +189,5 @@
   <!-- Base and Drive -->
   <gazebo reference="base_link">
-      <material>Gazebo/Gray</material>
+      <material>HelloRobot/LightGray</material>
   </gazebo>
   <gazebo reference="link_right_wheel">
@@ -91,5 +196,5 @@
       <kp value="10000000.0" />
       <kd value="100.0" />
-      <material>Gazebo/Blue</material>
+      <material>HelloRobot/Black</material>
       <minDepth>0.001</minDepth>
   </gazebo>
@@ -99,5 +204,5 @@
       <kp value="10000000.0" />
       <kd value="100.0" />
-      <material>Gazebo/Blue</material>
+      <material>HelloRobot/Black</material>
       <minDepth>0.001</minDepth>
   </gazebo>
@@ -105,5 +210,5 @@
     <turnGravityOff>false</turnGravityOff>
     <minDepth>0.001</minDepth>
-    <material>Gazebo/Blue</material>
+    <material>HelloRobot/Black</material>
     <mu1>0.0</mu1>
     <mu2>0.0</mu2>
@@ -128,84 +233,4 @@
 		</transmission>
   <!-- Sensors -->
-  <!-- Navigation camera -->
-  <gazebo reference="navigation_camera_link">
-    <sensor type="camera" name="navigation_camera">
-      <update_rate>6.0</update_rate>
-      <camera name="head">
-        <horizontal_fov>1.8</horizontal_fov>
-        <image>
-          <width>1024</width>
-          <height>768</height>
-          <format>R8G8B8</format>
-        </image>
-        <clip>
-          <near>0.02</near>
-          <far>100</far>
-        </clip>
-        <noise>
-          <type>gaussian</type>
-          <!-- Noise is sampled independently per pixel on each frame.
-               That pixel's noise value is added to each of its color
-               channels, which at that point lie in the range [0,1]. -->
-          <mean>0.0</mean>
-          <stddev>0.007</stddev>
-        </noise>
-      </camera>
-      <plugin name="camera_controller" filename="libgazebo_ros_camera.so">
-        <alwaysOn>false</alwaysOn>
-        <updateRate>0.0</updateRate>
-        <cameraName>navigation_camera</cameraName>
-        <imageTopicName>image_raw</imageTopicName>
-        <cameraInfoTopicName>camera_info</cameraInfoTopicName>
-        <frameName>camera_link</frameName>
-        <hackBaseline>0.07</hackBaseline>
-        <distortionK1>0.0</distortionK1>
-        <distortionK2>0.0</distortionK2>
-        <distortionK3>0.0</distortionK3>
-        <distortionT1>0.0</distortionT1>
-        <distortionT2>0.0</distortionT2>
-      </plugin>
-    </sensor>
-  </gazebo>
-  <!-- Gripper camera -->
-  <gazebo reference="gripper_camera_link">
-    <sensor type="camera" name="gripper_camera">
-      <update_rate>6.0</update_rate>
-      <camera name="head">
-        <horizontal_fov>1.8</horizontal_fov>
-        <image>
-          <width>1024</width>
-          <height>768</height>
-          <format>R8G8B8</format>
-        </image>
-        <clip>
-          <near>0.02</near>
-          <far>100</far>
-        </clip>
-        <noise>
-          <type>gaussian</type>
-          <!-- Noise is sampled independently per pixel on each frame.
-               That pixel's noise value is added to each of its color
-               channels, which at that point lie in the range [0,1]. -->
-          <mean>0.0</mean>
-          <stddev>0.007</stddev>
-        </noise>
-      </camera>
-      <plugin name="camera_controller" filename="libgazebo_ros_camera.so">
-        <alwaysOn>false</alwaysOn>
-        <updateRate>0.0</updateRate>
-        <cameraName>gripper_camera</cameraName>
-        <imageTopicName>image_raw</imageTopicName>
-        <cameraInfoTopicName>camera_info</cameraInfoTopicName>
-        <frameName>camera_link</frameName>
-        <hackBaseline>0.07</hackBaseline>
-        <distortionK1>0.0</distortionK1>
-        <distortionK2>0.0</distortionK2>
-        <distortionK3>0.0</distortionK3>
-        <distortionT1>0.0</distortionT1>
-        <distortionT2>0.0</distortionT2>
-      </plugin>
-    </sensor>
-  </gazebo>
   <xacro:if value="${'$(arg realsense)' == 'false' }">
     <gazebo reference="camera_depth_frame">
@@ -412,10 +437,10 @@
   <!-- Respeaker -->
   <gazebo reference="respeaker_base">
-      <material>Gazebo/Green</material>
+      <material>HelloRobot/Black</material>
   </gazebo>
   <!-- Non GPU LIDAR -->
   <xacro:unless value="$(arg gpu_lidar)">
     <gazebo reference="laser">
-      <material>Gazebo/Black</material>
+      <material>HelloRobot/Black</material>
       <sensor type="ray" name="laser_sensor">
         <pose>0 0 0 0 0 0</pose>
@@ -452,5 +477,5 @@
   <xacro:if value="$(arg gpu_lidar)">
     <gazebo reference="laser">
-      <material>Gazebo/Black</material>
+      <material>HelloRobot/Black</material>
       <sensor type="gpu_ray" name="laser_sensor">
         <pose>0 0 0 0 0 0</pose>
@@ -503,23 +528,4 @@
     </sensor>
   </gazebo>
-  <!-- Wrist IMU -->
-  <gazebo reference="link_wrist_yaw">
-    <gravity>true</gravity>
-    <sensor name="wrist_imu" type="imu">
-      <always_on>true</always_on>
-      <visualize>false</visualize>
-      <plugin name="imu_plugin" filename="libgazebo_ros_imu_sensor.so">
-        <topicName>wrist_imu/data</topicName>
-        <bodyName>link_wrist_yaw</bodyName>
-        <updateRateHZ>25.0</updateRateHZ>
-        <gaussianNoise>0.001</gaussianNoise>
-        <xyzOffset>0 0 0</xyzOffset>
-        <rpyOffset>0 0 0</rpyOffset>
-        <frameName>link_wrist_yaw</frameName>
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
Commit message: Update readme instructions for Stretch usage
Enable grasp hack on stretch grippers by default
Update a stretch part's material

File: robots/forky.gazebo.xacro (robot description, xacro)
@@ -662,5 +662,5 @@
       <kp value="10000000.0" />
       <kd value="100.0" />
-      <material>Gazebo/Gray</material>
+      <material>HelloRobot/Black</material>
       <minDepth>0.001</minDepth>
   </gazebo>

File: urdf/stretch_dex_wrist.gazebo.xacro (robot description, xacro)
@@ -107,5 +107,5 @@
       </joint>
     </transmission>
-    <!--gazebo>
+    <gazebo>
        <plugin name="gazebo_grasp_fix" filename="libgazebo_grasp_fix.so">
             <arm>
@@ -123,5 +123,5 @@
            <contact_topic>__default_topic__</contact_topic>
         </plugin>
-    </gazebo-->
+    </gazebo>
     <transmission name="trans_wrist_pitch">
       <type>transmission_interface/SimpleTransmission</type>

File: urdf/stretch_gripper.gazebo.xacro (robot description, xacro)
@@ -107,5 +107,5 @@
     </joint>
   </transmission>
-  <!--gazebo>
+  <gazebo>
      <plugin name="gazebo_grasp_fix" filename="libgazebo_grasp_fix.so">
           <arm>
@@ -123,5 +123,5 @@
          <contact_topic>__default_topic__</contact_topic>
       </plugin>
-  </gazebo-->
+  </gazebo>
     <gazebo>
       <plugin filename="libroboticsgroup_upatras_gazebo_mimic_joint_plugin.so" name="gripper_mimic1">
